File: FPGA_DevBoard/KiCAD_Files/Power.kicad_sch (KiCad schematic)
At the start: 65 parts, among them J10 Screw_Terminal_01x02, J11 Screw_Terminal_01x02, J12 Screw_Terminal_01x02, J13 Screw_Terminal_01x02, J4 USB4105-GF-A-060, J8 Screw_Terminal_01x02, Q1 IRF9358TRPBF, U16 MMSZ10T1G, U18 TPS62132RGTR, U3 CYPD3177-24LQXQT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

Commit message: Power Inductors
Parts:
- removed L1: 4.7u, Inductor_SMD:L_APV_ANR5020, symbol Device:L
- removed L2: 10u, Inductor_SMD:L_TechFuse_SL0624, symbol Device:L
- removed L3: 0.68u, Inductor_SMD:L_Sunlord_MWSA0402S, symbol Device:L
- removed L4: 2.2u, Inductor_SMD:L_Chilisin_BMRA00040415, symbol Device:L
- added L1: 4.7uH, FPGA_Power:IND-SMD_L7.4-W6.6, symbol FPGA_POWER:CKST0603-4.7UH/M_C3002636
- added L3: 680nH, FPGA_Power:IND-SMD_MPL-AL4020-R68, symbol FPGA_POWER:MPL-AL4020-R68
- added L4: 2.2uH, FPGA_Power:IND-SMD_L5.7-W5.2_CYA0530, symbol FPGA_POWER:CYA0530-2.2UH
- added U40: 10uH, FPGA_Power:IND-SMD_L6.0-W6.0_MPL-SE6040, symbol FPGA_POWER:MPL-SE6040-100
Connections:
- net +1V0: now also L3.2
- net +1V8: now also U40.2
- net +3V3: now also L4.1
- net +5V: now also L1.1
- net at U6.9 (SW): now also U40.1
- net at U18.1 (SW), U18.2 (SW), U18.3 (SW): now also L4.2
- net at R62.1, U5.7 (SW): now also L3.1
- net at C27.2, U4.5 (SW): now also L1.2

Commit message: OK I PULL UP
Added pull up resistors to SPI CS, pull down to GPIO12, redid vga bus lines. This also might include the FPGA clock being correct? Idk if that was committed before
Parts:
- removed J10, J11, J12, J13, J8: Screw_Terminal_01x02, FPGA_Interface:CONN-TH_2P-P5.00_CPC3703CTR, symbol Connector:Screw_Terminal_01x02

Commit message: Final Final Final Lol
Parts:
- added D10, D7, D8, D9: LED, Diode_SMD:D_0603_1608Metric, symbol Device:LED
- added R111, R114: 10k, Resistor_SMD:R_0603_1608Metric, symbol Device:R_US
- added R113, R115: 5k, Resistor_SMD:R_0603_1608Metric, symbol Device:R_US
Connections:
- net +1V0: now also R113.1
- net +1V8: now also R115.1
- net +3V3: now also R111.1
- net +5V: now also R114.1
- net GND: now also D10.1 (K), D7.1 (K), D8.1 (K), D9.1 (K)
- new net: D7.2 (A), R111.2
- new net: D10.2 (A), R115.2
- new net: D8.2 (A), R113.2
- new net: D9.2 (A), R114.2
