File: FPGA_DevBoard/KiCAD_Files/FPGA_UNIT_B.kicad_sch (KiCad schematic)
At the start: 82 parts, among them J15 6130XX11121_61301611121, J16 6130XX11121_61301611121, J7 L77HDE15SD1CH4F, U19 XC7S50-1FTGB196C, U21 USBLC6-2SC6, U22 USBLC6-2SC6, U23 USBLC6-2SC6, U24 USBLC6-2SC6, U25 USBLC6-2SC6, U26 USBLC6-2SC6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

Commit message: This is V2 Ordered
Parts:
- R31, R33: value 100 -> 200
Changed lines of the file:
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@@
 			)
 		)
-		(property "Value" "100"
+		(property "Value" "200"
 			(at 55.88 119.3799 0)
 			(show_name no)
@@
 			)
 		)
-		(property "Value" "100"
+		(property "Value" "200"
 			(at 46.99 105.4099 0)
 			(show_name no)
