File: FPGA_DevBoard/KiCAD_Files/USB_HUB.kicad_sch (KiCad schematic)
At the start: 26 parts, among them J5 USB-A1HSW6, J6 USB-A1HSW6, U11 MAX3421EETJ+T, U13 MAX3421EETJ+T, X3 12MHz, X4 12MHz

Commit message: Final Final Final Lol
Connections:
- net Max2_Int: now reaches U13.18 (INT)
- net GPIO_20: now reaches U13.28 (GPIN2)
- net Max1_Int: now reaches U11.18 (INT)
- no-connect marks 20 -> 19
Changed lines of the file:
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@@
-	)
-	(no_connect
-		(at 229.87 52.07)
 	)
 	(no_connect
@@
 	(wire
 		(pts
+			(xy 243.84 129.54) (xy 229.87 129.54)
+		)
+		(stroke
+			(width 0)
+			(type default)
+		)
+	)
+	(wire
+		(pts
 			(xy 163.83 120.65) (xy 179.07 120.65)
 		)
@@
 		(pts
 			(xy 157.48 102.87) (xy 179.07 102.87)
+		)
+		(stroke
+			(width 0)
+			(type default)
+		)
+	)
+	(wire
+		(pts
+			(xy 237.49 64.77) (xy 229.87 64.77)
 		)
 		(stroke
@@
 		)
 	)
+	(global_label "GPIO_20"
+		(shape input)
+		(at 229.87 52.07 0)
+		(fields_autoplaced yes)
+		(effects
+			(font
+				(size 1.27 1.27)
+			)
+			(justify left)
+		)
+		(property "Intersheetrefs" "${INTERSHEET_REFS}"
+			(at 240.7171 52.07 0)
+			(hide yes)
+			(show_name no)
+			(do_not_autoplace no)
+			(effects
+				(font
+					(size 1.27 1.27)
+				)
+				(justify left)
+			)
+		)
+	)
 	(global_label "GPIO_1"
 		(shape input)
@@
 		)
 	)
+	(global_label "Max2_Int"
+		(shape input)
+		(at 237.49 64.77 0)
+		(fields_autoplaced yes)
+		(effects
+			(font
+				(size 1.27 1.27)
+			)
+			(justify left)
+		)
+		(property "Intersheetrefs" "${INTERSHEET_REFS}"
+			(at 248.7603 64.77 0)
+			(hide yes)
+			(show_name no)
+			(do_not_autoplace no)
+			(effects
+				(font
+					(size 1.27 1.27)
+				)
+				(justify left)
+			)
+		)
+	)
 	(global_label "Max_SCLK_2"
 		(shape input)
@@
 			)
 		)
+	)
+	(global_label "Max1_Int"
+		(shape input)
+		(at 243.84 129.54 0)
+		(fields_autoplaced yes)
+		(effects
+			(font
+				(size 1.27 1.27)
+			)
+			(justify left)
+		)
+		(property "Intersheetrefs" "${INTERSHEET_REFS}"
+			(at 255.1103 129.54 0)
+			(hide yes)
+			(show_name no)
+			(do_not_autoplace no)
+			(effects
+				(font
+					(size 1.27 1.27)
+				)
+				(justify left)
+			)
+		)

Commit message: This is V2 Ordered
Parts:
- R11, R12, R13, R14: value 33 -> 33 +- 1%
Other:
- note added: "Copied from FTDI"
Changed lines of the file:
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@@
 		)
 	)
+	(text ""
+		(exclude_from_sim no)
+		(at 82.55 102.108 0)
+		(effects
+			(font
+				(size 2.54 2.54)
+			)
+		)
+	)
+	(text "Copied from FTDI"
+		(exclude_from_sim no)
+		(at 91.948 101.6 0)
+		(effects
+			(font
+				(size 2.54 2.54)
+			)
+		)
+	)
 	(text "USB ports, filtering for 5V\n"
 		(exclude_from_sim no)
@@
 	(wire
 		(pts
+			(xy 160.02 53.34) (xy 179.07 53.34)
+		)
+		(stroke
+			(width 0)
+			(type default)
+		)
+	)
+	(wire
+		(pts
 			(xy 35.56 96.52) (xy 35.56 99.06)
 		)
@@
 	(wire
 		(pts
-			(xy 160.02 53.34) (xy 179.07 53.34)
-		)
-		(stroke
-			(width 0)
-			(type default)
-		)
-	)
-	(wire
-		(pts
 			(xy 114.0728 162.56) (xy 127 162.56)
 		)
@@
 	)
 	(label "USB2+"
-		(at 172.72 55.88 180)
+		(at 179.07 55.88 180)
 		(effects
 			(font
@@
 	)
 	(label "USB2-"
-		(at 172.72 53.34 180)
+		(at 177.8 53.34 180)
 		(effects
 			(font
@@
 			)
 		)
-		(property "Value" "33"
-			(at 160.02 54.864 90)
+		(property "Value" "33 +- 1%"
+			(at 164.846 54.864 90)
 			(show_name no)
 			(do_not_autoplace no)
@@
 			)
 		)
-		(property "Value" "33"
-			(at 160.02 52.324 90)
+		(property "Value" "33 +- 1%"
+			(at 164.592 52.324 90)
 			(show_name no)
 			(do_not_autoplace no)
@@
 			)
 		)
-		(property "Value" "33"
-			(at 163.83 117.094 90)
+		(property "Value" "33 +- 1%"
+			(at 167.64 117.094 90)
 			(show_name no)
 			(do_not_autoplace no)
@@
 			)
 		)
-		(property "Value" "33"
-			(at 163.83 119.634 90)
+		(property "Value" "33 +- 1%"
+			(at 168.148 119.634 90)
 			(show_name no)
 			(do_not_autoplace no)
